File: hardware/protected_buck.kicad_pcb (KiCad board)
At the start: 2 copper layers, 120 x 70 mm, 32 parts, among them J1 VIN 8-18V, J2 5V OUT, J3 DAQ, U1 TPS26600PWP, U2 TPS5431DDA

Commit message: Improve hardware review and validation reporting
Parts:
- added R14: 0R, R_0603_1608Metric, F.Cu at (59.0, 91.0)
- added R15: 16.9k 1%, R_0603_1608Metric, F.Cu at (63.0, 91.0)
- added R16: 100k, R_0603_1608Metric, F.Cu at (69.0, 91.0)
- R6: value 10k -> 1k
Connections:
- C1 pad 2: GND -> RTN
- C2 pad 2: GND -> RTN
- C5 pad 2: GND -> RTN
- D1 pad 1: GND -> RTN
- J1 pad 2: GND -> RTN
- J3 pad 4: FLT -> FLT_DAQ
- J3 pad 6: IMON -> IMON_DAQ
- R2 pad 2: GND -> RTN
- R4 pad 2: GND -> RTN
- R5 pad 2: GND -> RTN
- R6 pad 1: PROTECTED_IN -> FLT
- R6 pad 2: FLT -> FLT_DAQ
- U1 pad 17: GND -> RTN
- U1 pad 6: GND -> MODE
- U1 pad 8: GND -> RTN
