File: hardware/protected_buck_unrouted.kicad_pcb (KiCad board)
At the start: 2 copper layers, 120 x 70 mm, 35 parts, among them J1 VIN 8-18V, J2 5V OUT, J3 DAQ, U1 TPS26600PWP, U2 TPS5431DDA

Commit message: Complete routed PCB and ERC-clean schematic
Routing:
- net VIN: track 159.3 -> 28.9 mm, vias 2 -> 0
- net SHDN: track 115.7 -> 0.00 mm, vias 2 -> 0
- net +5V: track 128.0 -> 25.8 mm, vias 2 -> 0
- net RTN: track 100.1 -> 0.00 mm, vias 4 -> 0
- net FLT_DAQ: track 74.5 -> 0.00 mm
- net IMON_DAQ: track 74.3 -> 0.00 mm
- net PROTECTED_IN: track 102.4 -> 56.9 mm, vias 1 -> 0
- net GND: track 36.7 -> 0.00 mm, vias 6 -> 0
- net OVP: track 34.0 -> 0.00 mm, vias 2 -> 0
- net VSENSE: track 32.6 -> 0.00 mm, vias 2 -> 0
- net IMON: track 30.4 -> 0.00 mm, vias 2 -> 0
- net UVLO: track 29.2 -> 0.00 mm, vias 2 -> 0
- net VOUT_SENSE: track 26.6 -> 0.00 mm
- net VIN_SENSE: track 22.8 -> 0.00 mm
- net FLT: track 16.5 -> 0.00 mm, vias 2 -> 0
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